File: transmitter/pcb/panel.kicad_pcb (KiCad board)
At the start: 2 copper layers, 30 x 118 mm, 4 parts, among them U1 3800, U3 M10_GPS_Module, U5 4754, U6 E22-400M30S

Commit message: Make receiver/transmitter firmware 'all' target auto-flash and add KiCad panel gerbers
- receiver/firmware/Makefile: 'make all' now builds and flashes (adds 'flash' dependency)
- transmitter/firmware/Makefile: 'make all' now compiles and flashes (adds 'flash' dependency)
- Add transmitter/pcb/outputs-new/ with panelized gerber files (gps-tracking-tx.zip + individual layers)
Routing:
- net Net-(U1-SCK/PA01): track 77.8 -> 73.6 mm, vias 1 -> 0
- net Net-(U1-D2/PA07): track 53.6 -> 49.3 mm, vias 1 -> 0
- net Net-(U1-MOSI/PA00): track 69.4 -> 65.3 mm, vias 1 -> 0
- net Net-(U1-MISO/PB23): track 61.4 -> 57.2 mm, vias 1 -> 0
- net Net-(U1-D12/PA23): track 79.8 -> 75.9 mm, vias 1 -> 0
Other:
- board size 30 x 118 mm -> 30 x 122.7 mm
Changed lines of the file:
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@@
       (drillshape 0)
       (scaleselection 1)
-      (outputdirectory "outputs/")
+      (outputdirectory "outputs-new/")
     )
   )
@@
       (net 2 "GND") (pinfunction "22-GND") (pintype "bidirectional") (solder_mask_margin 0.102))
   )
-  (gr_rect (start -15.0755 -59.1474) (end 14.9245 58.8526)
+  (gr_rect (start -15.0755 -63.821) (end 14.9245 58.8526)
     (stroke (width 0.05) (type default)) (fill none) (layer "Edge.Cuts"))
   (segment (start -11.5149 -23.8219) (end -11.5149 -21.2819) (width 1.2) (layer "F.Cu") (net 1))
@@
   (segment (start -12.5563 -18.7419) (end -12.6071 -18.6911) (width 0.8) (layer "F.Cu") (net 2))
   (via (at 12.9707 -49.1457) (size 1.7) (drill 1) (layers "F.Cu" "B.Cu") (net 2))
-  (via (at -0.0755 -55.1474) (size 6) (drill 5) (layers "F.Cu" "B.Cu") (free) (net 2))
-  (via (at 10.4245 54.8526) (size 6) (drill 5) (layers "F.Cu" "B.Cu") (free) (net 2))
+  (via (at 0 -59) (size 6) (drill 2) (layers "F.Cu" "B.Cu") (free) (net 2))
+  (via (at 10.5 55) (size 6) (drill 2) (layers "F.Cu" "B.Cu") (free) (net 2))
   (via (at -12.6071 -18.6911) (size 1.7) (drill 1) (layers "F.Cu" "B.Cu") (net 2))
-  (via (at -10.5755 54.8526) (size 6) (drill 5) (layers "F.Cu" "B.Cu") (free) (net 2))
+  (via (at -10.5 55) (size 6) (drill 2) (layers "F.Cu" "B.Cu") (free) (net 2))
   (via (at 13.0469 -18.6911) (size 1.7) (drill 1) (layers "F.Cu" "B.Cu") (net 2))
   (via (at 13.0469 -44.1673) (size 1.7) (drill 1) (layers "F.Cu" "B.Cu") (net 2))
@@
   (via (at -12.7341 -36.5219) (size 1.7) (drill 1) (layers "F.Cu" "B.Cu") (net 2))
   (segment (start 10.3451 23.1902) (end 10.3197 23.2156) (width 0.6) (layer "F.Cu") (net 3))
-  (segment (start 12.4533 23.1902) (end 10.3451 23.1902) (width 0.6) (layer "F.Cu") (net 3))
   (segment (start 0.0835 18.4404) (end 0.0835 -25.1206) (width 0.6) (layer "F.Cu") (net 3))
   (segment (start 0.0835 -29.0068) (end 5.0586 -33.9819) (width 0.6) (layer "F.Cu") (net 3))
@@
   (segment (start 0.0835 -29.0068) (end 0.0835 -25.1206) (width 0.6) (layer "F.Cu") (net 3))
   (segment (start 10.3197 23.2156) (end 4.8587 23.2156) (width 0.6) (layer "F.Cu") (net 3))
-  (via (at 12.4533 23.1902) (size 1.7) (drill 1) (layers "F.Cu" "B.Cu") (net 3))
   (segment (start 10.3451 23.1902) (end 10.3197 23.2156) (width 0.4) (layer "B.Cu") (net 3))
-  (segment (start 12.4533 23.1902) (end 10.3451 23.1902) (width 0.6) (layer "B.Cu") (net 3))
   (segment (start 2.2171 -27.3812) (end 2.2171 16.5862) (width 0.6) (layer "F.Cu") (net 4))
   (segment (start 2.2171 16.5862) (end 6.3065 20.6756) (width 0.6) (layer "F.Cu") (net 4))
   (segment (start 10.3705 20.6248) (end 10.3197 20.6756) (width 0.6) (layer "F.Cu") (net 4))
-  (segment (start 12.4533 20.6248) (end 10.3705 20.6248) (width 0.6) (layer "F.Cu") (net 4))
   (segment (start 6.3065 20.6756) (end 10.3197 20.6756) (width 0.6) (layer "F.Cu") (net 4))
   (segment (start 6.2778 -31.4419) (end 2.2171 -27.3812) (width 0.6) (layer "F.Cu") (net 4))
   (segment (start 11.8851 -31.4419) (end 6.2778 -31.4419) (width 0.6) (layer "F.Cu") (net 4))
-  (via (at 12.4533 20.6248) (size 1.7) (drill 1) (layers "F.Cu" "B.Cu") (net 4))
-  (segment (start 12.4533 20.6248) (end 10.3705 20.6248) (width 0.6) (layer "B.Cu") (net 4))
   (segment (start 10.3705 20.6248) (end 10.3197 20.6756) (width 0.4) (layer "B.Cu") (net 4))
   (segment (start 4.4523 -26.162) (end 4.4523 -22.2758) (width 0.6) (layer "F.Cu") (net 8))
@@
   (segment (start 4.4523 15.2146) (end 4.4523 -22.2758) (width 0.6) (layer "F.Cu") (net 8))
   (segment (start 4.4523 -26.162) (end 7.1922 -28.9019) (width 0.6) (layer "F.Cu") (net 8))
-  (segment (start 12.4533 18.0594) (end 10.3959 18.0594) (width 0.6) (layer "F.Cu") (net 8))
-  (via (at 12.4533 18.0594) (size 1.7) (drill 1) (layers "F.Cu" "B.Cu") (net 8))
-  (segment (start 12.4533 18.0594) (end 10.3959 18.0594) (width 0.6) (layer "B.Cu") (net 8))
   (segment (start 10.3959 18.0594) (end 10.3197 18.1356) (width 0.4) (layer "B.Cu") (net 8))
   (segment (start -7.0793 15.5956) (end -4.9203 15.5956) (width 0.6) (layer "B.Cu") (net 15))
@@
   (segment (start -4.9457 38.481) (end -4.9203 38.4556) (width 0.6) (layer "F.Cu") (net 26))
   (segment (start -1.9485 36.9316) (end -3.4725 38.4556) (width 0.6) (layer "F.Cu") (net 26))
-  (segment (start -6.9015 38.481) (end -4.9457 38.481) (width 0.6) (layer "F.Cu") (net 26))
   (segment (start -1.9485 -23.3426) (end -1.9485 36.9316) (width 0.6) (layer "F.Cu") (net 26))
   (segment (start -7.5078 -28.9019) (end -1.9485 -23.3426) (width 0.6) (layer "F.Cu") (net 26))
-  (via (at -6.9015 38.481) (size 1.7) (drill 1) (layers "F.Cu" "B.Cu") (net 26))
-  (segment (start -6.9015 38.481) (end -4.9457 38.481) (width 0.6) (layer "B.Cu") (net 26))
   (segment (start -4.9457 38.481) (end -4.9203 38.4556) (width 0.4) (layer "B.Cu") (net 26))
   (segment (start 6.6113 13.9192) (end 8.2877 15.5956) (width 0.6) (layer "F.Cu") (net 27))
@@
   (segment (start 8.2877 15.5956) (end 10.3197 15.5956) (width 0.6) (layer "F.Cu") (net 27))
   (segment (start 6.6113 -21.3106) (end 6.6113 13.9192) (width 0.6) (layer "F.Cu") (net 27))
-  (segment (start 12.4533 15.5702) (end 10.3451 15.5702) (width 0.6) (layer "F.Cu") (net 27))
-  (via (at 12.4533 15.5702) (size 1.7) (drill 1) (layers "F.Cu" "B.Cu") (net 27))
-  (segment (start 12.4533 15.5702) (end 10.3451 15.5702) (width 0.6) (layer "B.Cu") (net 27))
   (segment (start 10.3451 15.5702) (end 10.3197 15.5956) (width 0.4) (layer "B.Cu") (net 27))
   (zone (net 2) (net_name "GND") (layer "B.Cu") (hatch edge 0.6)
